File: Hardware/KiCAD/BHOA/amp.kicad_sch (KiCad schematic)
At the start: 20 parts, among them U1 OPA1688

Commit message: added outpout relays
Other:
- company: ncAudio -> C Audio
- title: NCBalOPHeadAmp -> BHOA
Changed lines of the file:
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@@
 (kicad_sch (version 20230121) (generator eeschema)
-  (paper "A5")
+  (paper "A4")
   (title_block
-    (title "NCBalOPHeadAmp")
+    (title "BHOA")
     (date "2023-10-31")
     (rev "0.1")
-    (company "ncAudio")
+    (company "C Audio")
+    (comment 3 "Balanced Headphone Operationsal Amplifier")
     (comment 4 "Paralleled OPAMP outputs for more power and lower distortion")
   )
