File: Hardware/KiCAD/BHOA/amp.kicad_sch (KiCad schematic)
At the start: 20 parts, among them U1 OPA1688

Commit message: Updated PCB with output protection
Parts:
- renumbered C100 to C70, C104 to C71, C101 to C72, C105 to C73, C102 to C74, C106 to C75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
