File: Hardware/KiCAD/BHOA/amp.kicad_sch (KiCad schematic)
At the start: 20 parts, among them U1 OPA1688

Commit message: added schematic pic
Parts:
- renumbered U1 to U100, U1 to U101, U1 to U102, U1 to U103
