File: Hardware/KiCAD/BHOA/input_filter.kicad_sch (KiCad schematic)
At the start: 5 parts

Commit message: added schematic pic
Parts:
- renumbered C2 to C801, C3 to C802, C4 to C803, R1 to R801, R8 to R802
